File: C64 Replacement PSU (230V)/Rev. 2/Eagle/C64_PS.brd (EAGLE design)
At the start: 134 x 70 mm, 33 parts, among them IC1 TSR2-2450

Commit message: Silk Screen Update
Parts:
- added U$17: OPEN_SOURCE_HW, Logo:OPENHW
- moved U$15 8.93 mm to (46.2, 1.11)
Other:
- board text added: "100n"
- board text added: "10n/ 500V"
- board text added: "1M"
- board text added: "1N 4007"
- board text added: "1N 5908"
- board text added: "2200u/50V"
- board text added: "47u"
- board text added: "50V"
- board text added: "B32922C3334M"
- board text added: "KBU404"
- board text added: "P6KE15CA"
- board text added: "TSR2-2450"
- board text added: "for LED"
- board text added: "http://github.com/ svenpetersen1965"
